Commit message: feat: ros nodes for black and white able to play against each other; moveit + ompl not fully implemented

File: src/chess_robot_description/urdf/dual_fr3.urdf.xacro (robot description, xacro)
@@ -1,77 +1,55 @@
 <?xml version="1.0"?>
 <robot xmlns:xacro="http://www.ros.org/wiki/xacro" name="dual_fr3">
-  <!--
-    Dual FR3 setup. White on the rank 1-2 side (low world X). Black on the
-    rank 7-8 side (high world X), yawed 180 deg to face white.
-    With gazebo=true and connected_to=base (default), the franka_robot macro
-    skips emitting a parent link/joint, so we wire each arm's link0 to world
-    ourselves with the offsets below.
-    ros2_control on franka_robot is left false because upstream's bundled
-    franka_arm.ros2_control.xacro emits the gz_ros2_control system plugin
-    once per call (-> two controller_managers under dual-arm) and hardcodes
-    its `<parameters>` to `franka_gazebo_bringup` (not packaged for Humble).
-    Instead we include our forked franka_arm.ros2_control.xacro and call its
-    macro twice ourselves: white emits the plugin pointing at our YAML,
-    black skips the plugin emission.
-  -->
   <xacro:arg name="white_xyz" default="-0.5 0 0.75"/>
-  <xacro:arg name="white_rpy" default="0 0 0"/>
   <xacro:arg name="black_xyz" default="0.5 0 0.75"/>
-  <xacro:arg name="black_rpy" default="0 0 3.14159265359"/>
-  <xacro:arg name="controllers_yaml" default="$(find chess_robot_description)/config/fr3_controllers.yaml"/>
-  <xacro:include filename="$(find franka_description)/robots/common/franka_robot.xacro"/>
+  <xacro:include filename="$(find franka_description)/robots/common/franka_arm.xacro"/>
+  <xacro:include filename="$(find franka_description)/end_effectors/common/utils.xacro"/>
+  <xacro:include filename="$(find franka_description)/end_effectors/common/franka_hand.xacro"/>
   <xacro:include filename="$(find chess_robot_description)/urdf/franka_arm.ros2_control.xacro"/>
-  <link name="world"/>
-  <!-- White arm body (no ros2_control here; we add our forked one below) -->
-  <xacro:franka_robot
+  <!-- White arm: attached to world -->
+  <xacro:franka_arm
       robot_type="fr3"
       arm_prefix="white_"
-      joint_limits="${xacro.load_yaml('$(find franka_description)/robots/fr3/joint_limits.yaml')}"
-      inertials="${xacro.load_yaml('$(find franka_description)/robots/fr3/inertials.yaml')}"
-      kinematics="${xacro.load_yaml('$(find franka_description)/robots/fr3/kinematics.yaml')}"
-      accelerometer_config="${xacro.load_yaml('$(find franka_description)/robots/fr3/accelerometers.yaml')}"
-      dynamics="${xacro.load_yaml('$(find franka_description)/robots/fr3/dynamics.yaml')}"
-      hand="true"
-      ee_id="franka_hand"
-      gazebo="true"
-      ros2_control="false"/>
-  <joint name="world_to_white_arm" type="fixed">
-    <parent link="world"/>
-    <child link="white_fr3_link0"/>
-    <origin xyz="$(arg white_xyz)" rpy="$(arg white_rpy)"/>
+      connected_to="world"
+      xyz="$(arg white_xyz)"
+      rpy="0 0 0"
+      gazebo="true" />
+  <!-- Black arm: no connected_to to avoid re-declaring white_fr3_link0 -->
+  <xacro:franka_arm
+      robot_type="fr3"
+      arm_prefix="black_"
+      connected_to=""
+      xyz="0 0 0"
+      rpy="0 0 0"
+      gazebo="true" />
+  <!-- Manually attach black_fr3_link0 to white_fr3_link0 -->
+  <joint name="white_to_black_base_joint" type="fixed">
+    <parent link="white_fr3_link0"/>
+    <child link="black_fr3_link0"/>
+    <origin xyz="1.0 0 0" rpy="0 0 3.14159"/>
   </joint>
+  <xacro:franka_hand
+      robot_type="fr3"
+      arm_prefix="white_"
+      connected_to="white_fr3_link8"
+      ee_id="franka_hand_white"
+      ee_inertials="${xacro.load_yaml('$(find franka_description)/end_effectors/franka_hand/inertials.yaml')}"
+      gazebo="true" />
   <xacro:franka_arm_ros2_control
-      robot_type="fr3"
-      robot_ip=""
       arm_prefix="white_"
       gazebo="true"
-      hand="true"
       emit_gazebo_plugin="true"
-      controllers_yaml="$(arg controllers_yaml)"/>
-  <!-- Black arm body -->
-  <xacro:franka_robot
+      controllers_yaml="$(find chess_robot_description)/config/fr3_controllers.yaml"/>
+  <xacro:franka_hand
       robot_type="fr3"
       arm_prefix="black_"
-      joint_limits="${xacro.load_yaml('$(find franka_description)/robots/fr3/joint_limits.yaml')}"
-      inertials="${xacro.load_yaml('$(find franka_description)/robots/fr3/inertials.yaml')}"
-      kinematics="${xacro.load_yaml('$(find franka_description)/robots/fr3/kinematics.yaml')}"
-      accelerometer_config="${xacro.load_yaml('$(find franka_description)/robots/fr3/accelerometers.yaml')}"
-      dynamics="${xacro.load_yaml('$(find franka_description)/robots/fr3/dynamics.yaml')}"
-      hand="true"
-      ee_id="franka_hand"
-      gazebo="true"
-      ros2_control="false"/>
-  <joint name="world_to_black_arm" type="fixed">
-    <parent link="world"/>
-    <child link="black_fr3_link0"/>
-    <origin xyz="$(arg black_xyz)" rpy="$(arg black_rpy)"/>
-  </joint>
+      connected_to="black_fr3_link8"
+      ee_id="franka_hand_black"
+      ee_inertials="${xacro.load_yaml('$(find franka_description)/end_effectors/franka_hand/inertials.yaml')}"
+      gazebo="true" />
   <xacro:franka_arm_ros2_control
-      robot_type="fr3"
-      robot_ip=""
       arm_prefix="black_"
       gazebo="true"
-      hand="true"
       emit_gazebo_plugin="false"
-      controllers_yaml="$(arg controllers_yaml)"/>
+      controllers_yaml="$(find chess_robot_description)/config/fr3_controllers.yaml"/>
 </robot>

File: src/chess_robot_description/urdf/franka_arm.ros2_control.xacro (robot description, xacro)
@@ -1,19 +1,8 @@
 <?xml version="1.0"?>
-<!--
-  Fork of franka_description/robots/common/franka_arm.ros2_control.xacro
-  (verified against frankarobotics/franka_description@2.6.0).
-  Two changes from upstream:
-    * `controllers_yaml` param replaces the hardcoded
-      `$(find franka_gazebo_bringup)/config/franka_gazebo_controllers.yaml`,
-      which depends on a package not packaged for Humble.
-    * `emit_gazebo_plugin` param gates the gz_ros2_control system plugin so
-      it's only emitted on one of multiple macro invocations (one
-      controller_manager total across both arms).
-  Everything else is byte-identical to upstream.
--->
 <robot xmlns:xacro="http://www.ros.org/wiki/xacro">
 <xacro:macro name="franka_arm_ros2_control"
-         params="robot_type
-                 robot_ip
+         params="arm_prefix
+                 robot_type:='fr3'
+                 robot_ip:=''
                  use_fake_hardware:=false
                  fake_sensor_commands:=false
@@ -21,32 +10,18 @@
                  hand:=false
                  gazebo_effort:=false
-                 arm_prefix:=''
                  is_async:=false
                  thread_priority:=50
                  emit_gazebo_plugin:=true
-                 controllers_yaml:='$(find chess_robot_description)/config/fr3_controllers.yaml'">
+                 controllers_yaml">
     <ros2_control name="${arm_prefix}FrankaHardwareInterface" type="system" is_async="${is_async}">
-        <xacro:if value="${is_async}">
-          <properties>
-            <async scheduling_policy="detached" print_warnings="true" thread_priority="${thread_priority}" manage_overruns="false"/>
-          </properties>
-        </xacro:if>
         <hardware>
-          <param name="version">1.0.0</param>
           <param name="robot_type">${robot_type}</param>
-          <param name="prefix">${arm_prefix}</param>
-          <xacro:if value="${use_fake_hardware}">
-            <plugin>mock_components/GenericSystem</plugin>
-            <param name="fake_sensor_commands">${fake_sensor_commands}</param>
-            <param name="state_following_offset">0.0</param>
-          </xacro:if>
           <xacro:if value="${gazebo}">
             <plugin>gz_ros2_control/GazeboSimSystem</plugin>
           </xacro:if>
-          <xacro:if value="${use_fake_hardware == 0 and gazebo == 0}">
+          <xacro:unless value="${gazebo}">
             <plugin>franka_hardware/FrankaHardwareInterface</plugin>
             <param name="robot_ip">${robot_ip}</param>
-            <param name="arm_prefix">${arm_prefix}</param>
-          </xacro:if>
+          </xacro:unless>
         </hardware>
       <xacro:macro name="configure_joint" params="joint_name initial_position">
@@ -54,13 +29,8 @@
             <command_interface name="position"/>
             <command_interface name="velocity"/>
-          <xacro:if value="${gazebo == 0 or gazebo_effort == 1}">
-            <command_interface name="effort"/>
-          </xacro:if>
-          <state_interface name="position">
-            <param name="initial_value">${initial_position}</param>
-          </state_interface>
-          <state_interface name="velocity"/>
-            <param name="initial_value">0.0</param>
-          <state_interface name="effort"/>
+            <state_interface name="position">
+              <param name="initial_value">${initial_position}</param>
+            </state_interface>
+            <state_interface name="velocity"/>
         </joint>
       </xacro:macro>
@@ -75,25 +45,4 @@
         <xacro:configure_joint joint_name="${arm_prefix}${robot_type}_finger_joint1" initial_position="0.0" />
       </xacro:if>
-      <xacro:macro name="general_purpose_io" params="prefix command_interface index">
-        <gpio name="${arm_prefix}${prefix}">
-          <command_interface name="${command_interface}"/>
-          <param name="index">${index}</param>
-        </gpio>
-      </xacro:macro>
-      <xacro:general_purpose_io prefix="vx" command_interface="cartesian_velocity" index="0"/>
-      <xacro:general_purpose_io prefix="vy" command_interface="cartesian_velocity" index="1"/>
-      <xacro:general_purpose_io prefix="vz" command_interface="cartesian_velocity" index="2"/>
-      <xacro:general_purpose_io prefix="wx" command_interface="cartesian_velocity" index="3"/>
-      <xacro:general_purpose_io prefix="wy" command_interface="cartesian_velocity" index="4"/>
-      <xacro:general_purpose_io prefix="wz" command_interface="cartesian_velocity" index="5"/>
-      <xacro:macro name="loop" params="i">
-        <xacro:unless value="${i == 16}">
-          <xacro:general_purpose_io prefix="${i}" command_interface="cartesian_pose_command" index="${i}"/>
-          <xacro:loop i="${i+1}"/>
-        </xacro:unless>
-      </xacro:macro>
-      <xacro:loop i="0"/>
-      <xacro:general_purpose_io prefix="joint_3_position" command_interface="elbow_command" index="0"/>
-      <xacro:general_purpose_io prefix="joint_4_sign" command_interface="elbow_command" index="1"/>
     </ros2_control>
     <xacro:if value="${gazebo and emit_gazebo_plugin}">
@@ -101,4 +50,5 @@
         <plugin filename="gz_ros2_control-system" name="gz_ros2_control::GazeboSimROS2ControlPlugin">
           <parameters>${controllers_yaml}</parameters>
+          <use_sim_time>false</use_sim_time>
         </plugin>
       </gazebo>
